File: ACDC_Convertor/ACDC_Convertor.kicad_pcb (KiCad board)
At the start: 2 copper layers, 38.1 x 30.5 mm, 6 parts, among them J1 Screw_Terminal_01x02, J2 Screw_Terminal_01x02, U1 0433BM15A0001, U2 L78L12_SO8

Commit message: feat:new projects
Parts:
- moved J2 5.80 mm to (118.7, 103.9), turned to 0 degrees
Routing:
- net Net-(C1-Pad2): track 0.00 -> 50.2 mm
- net Net-(J1-Pad1): track 0.00 -> 40.8 mm
- net Net-(C1-Pad1): track 0.00 -> 34.6 mm
- net Net-(J1-Pad2): track 0.00 -> 29.1 mm
- net Net-(D1-Pad2): track 0.00 -> 28.3 mm
- net Net-(D1-Pad3): track 0.00 -> 16.9 mm
- net Net-(J2-Pad1): track 0.00 -> 13.8 mm
