File: MosquitoRepellant/MosquitoRepellant.kicad_pcb (KiCad board)
At the start: 2 copper layers, 48.8 x 44.8 mm, 11 parts, among them U1 NE555D

Commit message: feat:new projects
Connections:
- net Net-(BT1-+) renamed +5V
- net Net-(BT1--) renamed GND
Routing:
- net +5V: track 0.00 -> 50.4 mm
- net Net-(R2-Pad2): track 0.00 -> 21.9 mm
- net Net-(U1-THR): track 12.3 -> 33.2 mm, vias 0 -> 1
- net Net-(BZ1-+): track 0.00 -> 20.4 mm
- net Net-(U1-DIS): track 0.00 -> 19.4 mm
- net GND: track 19.2 -> 36.2 mm, vias 0 -> 1
- added copper zone on F.Cu, net +5V
- added copper zone on B.Cu, net GND
