File: MosquitoRepellant/MosquitoRepellant.kicad_pcb (KiCad board)
At the start: 2 copper layers, 48.8 x 44.8 mm, 11 parts, among them U1 NE555D

Commit message: ods:Mosquito project
Routing:
- net Net-(BT1-+): track 0.00 -> 56.5 mm
- net Net-(R2-Pad2): track 0.00 -> 29.2 mm
- net Net-(BZ1-+): track 0.00 -> 20.1 mm, vias 0 -> 1
- net Net-(U1-DIS): track 0.00 -> 19.4 mm
- net Net-(U1-THR): track 12.3 -> 29.7 mm, vias 0 -> 1
- net Net-(BT1--): track 19.2 -> 34.1 mm
