File: School Projects/Chaser Board/Chaser Board.kicad_sch (KiCad schematic)
At the start: 22 parts, among them U1 ATmega328-P, Y1 Crystal

Commit message: added prod of chaser board,updates to car battery detector and started simple power supply project
Parts:
- added H1, H2, H3, H4: MountingHole, MountingHole:MountingHole_2.5mm_Pad_Via, symbol Mechanical:MountingHole
- C1, C2, Creset1: footprint (none) -> Capacitor_SMD:C_0805_2012Metric
- D1, D2, D3, D4, D5, D6, D7, D8: footprint (none) -> LED_THT:LED_D5.0mm
- R1, R2, R3, R4, R5, R6, R7, R8: footprint (none) -> Resistor_THT:R_Axial_DIN0204_L3.6mm_D1.6mm_P5.08mm_Horizontal
- Rreset1: footprint (none) -> Resistor_SMD:R_0805_2012Metric_Pad1.20x1.40mm_HandSolder
- Y1: footprint (none) -> Crystal:Crystal_HC49-4H_Vertical
Other:
- note added: "Mounting Hole"
