File: School Projects/Simple Power Supply Board/Simple_power_supply_board/Simple_power_supply_board.kicad_sch (KiCad schematic)
At the start: 21 parts, among them J1 Barrel_Jack, J2 Screw_Terminal_01x02, J3 Screw_Terminal_01x02, U1 L7805, U3 MCP1700x-120xxMB

Commit message: added prod of simple power supply project
Parts:
- removed F1: 500mA / 1A, symbol Device:Polyfuse
- removed U1: L7805, symbol Regulator_Linear:L7805
- added H1, H2, H3, H4: MountingHole, MountingHole:MountingHole_2.2mm_M2_DIN965_Pad_TopOnly, symbol Mechanical:MountingHole
- added U1: PTC_FUSE, Fuse:PTC_FUSE, symbol PTC_FUSE:RUEF300
- added U2: LD1117V50, Package_TO_SOT_THT:TO-220-3_Vertical, symbol Regulator_Linear:LD1117V50
- J1: renamed from J3; footprint (none) -> TerminalBlock_Phoenix:TerminalBlock_Phoenix_MKDS-1,5-2-5.08_1x02_P5.08mm_Horizontal
- J2: footprint (none) -> TerminalBlock_Phoenix:TerminalBlock_Phoenix_MKDS-1,5-2-5.08_1x02_P5.08mm_Horizontal
- J3: renamed from J1; footprint (none) -> Connector_BarrelJack:BarrelJack_GCT_DCJ200-10-A_Horizontal
- R1, R2: footprint (none) -> Resistor_THT:R_Axial_DIN0309_L9.0mm_D3.2mm_P12.70mm_Horizontal
- renumbered C3 to C1, C4 to C3, C1 to C4, C7 to C5, C5 to C6, C8 to C7, C6 to C8, D4 to D3, D5 to D4, D3 to D5
Connections:
- net 5V: now also U2.2 (VO)
- net GND: now also U2.1 (GND)
- net VR: now also U1.P$2, U2.3 (VI)
- net at D1.1 (K): now also U1.P$1
Other:
- note added: "MOUNT HOLES"
- moved on the sheet: D1
