File: School Projects/Sensor and Display Module/Sensor and Display Module.kicad_pcb (KiCad board)
At the start: 2 copper layers, 64.3 x 88.9 mm, 27 parts, among them U1 ATmega328-P

Commit message: mods to display sensor module pcb routing
Parts:
- moved U1 33.3 mm to (88.9, 115.5), turned to 90 degrees
- turned MUX1 to -90 degrees
Routing:
- net +5V: track 231.5 -> 299.3 mm, vias 13 -> 8
- net /RST: track 62.7 -> 104.5 mm, vias 1 -> 2
- net /SC1: track 61.6 -> 27.3 mm
- net /SDA: track 84.2 -> 116.5 mm, vias 9 -> 3
- net /SCL: track 74.1 -> 102.9 mm, vias 9 -> 3
- net /SD1: track 55.8 -> 31.9 mm
- net /SC2: track 43.2 -> 20.2 mm
- net /SD2: track 39.2 -> 19.4 mm
- net GND: track 294.5 -> 313.0 mm, vias 10 -> 6
- net /SD4: track 28.3 -> 10.6 mm, vias 2 -> 0
- net /SC4: track 28.6 -> 12.1 mm, vias 2 -> 0
- net /SC3: track 25.7 -> 11.1 mm, vias 2 -> 0
- net /SD5: track 32.7 -> 18.3 mm
- net /SD3: track 24.5 -> 12.1 mm, vias 2 -> 0
- net /SC5: track 30.3 -> 18.4 mm
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- removed copper zone on F.Cu, net +5V
- removed copper zone on F.Cu, net GND
