File: School Projects/ESP32 Dev Board Clone/ESP32 Dev Board Clone/ESP32 Dev Board Clone.kicad_sch (KiCad schematic)
At the start: 25 parts, among them J1 Conn_01x03_Pin, J3 Barrel_Jack, P1 USB_C_Plug_USB2.0, U1 ESP32-WROOM-32, U2 CP2102N-Axx-xQFN24, U3 AMS1117-3.3

Commit message: yet to assign footprints in next commit
Parts:
- removed R3, R4: 4.7KΩ, Resistor_THT:R_Axial_DIN0207_L6.3mm_D2.5mm_P15.24mm_Horizontal, symbol Device:R_US
- added J2: Conn_01x06_Pin, symbol Connector:Conn_01x06_Pin
- added J4: Conn_01x03_Pin, symbol Connector:Conn_01x03_Pin
- added J5, J6: Conn_01x11_Pin, symbol Connector:Conn_01x11_Pin
- added R8, R9: 10KΩ, Resistor_THT:R_Axial_DIN0207_L6.3mm_D2.5mm_P15.24mm_Horizontal, symbol Device:R_US
- C1: value 10nF -> 100nF
Connections:
- net RTS is gone; now on net DTR_EN: C1.1, U1.3 (EN)
- net 3.3V: now also J2.1 (Pin_1), J4.2 (Pin_2), R8.1, R9.1; no longer C2.1, D1.2 (A), U3.2 (VO)
- net GND: now also J2.6 (Pin_6), J6.11 (Pin_11)
- net RX: now also J2.2 (Pin_2)
- net TX: now also J2.3 (Pin_3)
- net DA2C_IO1: now reaches U1.10 (IO25)
- net DA2C_IO1: now also J6.8 (Pin_8)
- net DA2C_IO2: now reaches U1.11 (IO26)
- net DA2C_IO2: now also J6.9 (Pin_9)
- net DA2T_IO3: now reaches U1.12 (IO27)
- net DA2T_IO3: now also J6.7 (Pin_7)
- net DA2T_IO2: now reaches U1.13 (IO14)
- net DA2T_IO2: now also J6.6 (Pin_6)
- net DA2T_IO1: now reaches U1.16 (IO13)
- net DA2T_IO1: now also J6.5 (Pin_5)
- net DA2T_IO0: now reaches U1.26 (IO4)
- net DA2T_IO0: now also J6.4 (Pin_4)
- net D_IO0: now reaches U1.27 (IO16)
- net D_IO0: now also J5.2 (Pin_2)
- net D_IO1: now reaches U1.28 (IO17)
- net D_IO1: now also J5.3 (Pin_3)
- net D_IO2: now reaches U1.30 (IO18)
- net D_IO2: now also J5.4 (Pin_4)
- net D_IO3: now reaches U1.31 (IO19)
- net D_IO3: now also J5.5 (Pin_5)
- net D_IO6: now reaches U1.37 (IO23)
- net D_IO6: now also J5.8 (Pin_8)
- net DA1_I2: now reaches U1.4 (SENSOR_VP)
- net DA1_I2: now also J6.2 (Pin_2)
- net DA1_I3: now reaches U1.5 (SENSOR_VN)
- net DA1_I3: now also J6.3 (Pin_3)
- net DA1_I0: now reaches U1.6 (IO34)
- net DA1_I0: now also J5.11 (Pin_11)
- net DA1_I1: now reaches U1.7 (IO35)
- net DA1_I1: now also J6.1 (Pin_1)
- net DA1T_IO0: now reaches U1.8 (IO32)
- net DA1T_IO0: now also J5.9 (Pin_9)
- net DA1T_IO1: now reaches U1.9 (IO33)
- net DA1T_IO1: now also J5.10 (Pin_10)
- net DTR renamed DTR_EN
- net DTR_EN: now also J2.4 (Pin_4), R8.2; no longer U1.25 (IO0)
- net EN renamed RTS_IO0
- net RTS_IO0: now also U1.25 (IO0), J2.5 (Pin_5), R9.2
- net SCL renamed D_IO5
- net D_IO5: now also J5.7 (Pin_7)
- net SDA renamed D_IO4
- net D_IO4: now also J5.6 (Pin_6)
- new net Ext3.3V: J4.3 (Pin_3), J5.1 (Pin_1)
- new net Vcc3.3V: C2.1, D1.2 (A), J4.1 (Pin_1), U3.2 (VO)
- no-connect marks 12 -> 23
Other:
- note added: "BreakOut Pins"
- note added: "Programming Header"
- moved on the sheet: C1, C9, J1

Commit message: Final parts of esp32 board
Parts:
- removed J1: Conn_01x03_Pin, Connector_PinHeader_2.54mm:PinHeader_1x03_P2.54mm_Vertical, symbol Connector:Conn_01x03_Pin
- removed J4: Conn_01x03_Pin, symbol Connector:Conn_01x03_Pin
- removed J5, J6: Conn_01x11_Pin, symbol Connector:Conn_01x11_Pin
- added H1: D_IO0, MountingHole:MountingHole_2.2mm_M2_DIN965_Pad_TopBottom, symbol Mechanical:MountingHole_Pad
- added H10: DA1T_IO1, MountingHole:MountingHole_2.2mm_M2_DIN965_Pad_TopBottom, symbol Mechanical:MountingHole_Pad
- added H11: DA1_I0, MountingHole:MountingHole_2.2mm_M2_DIN965_Pad_TopBottom, symbol Mechanical:MountingHole_Pad
- added H12: NC, MountingHole:MountingHole_2.2mm_M2_DIN965_Pad_TopBottom, symbol Mechanical:MountingHole_Pad
- added H13: DA2C_IO1, MountingHole:MountingHole_2.2mm_M2_DIN965_Pad_TopBottom, symbol Mechanical:MountingHole_Pad
- added H14: DA2T_IO2, MountingHole:MountingHole_2.2mm_M2_DIN965_Pad_TopBottom, symbol Mechanical:MountingHole_Pad
- added H15: DA2T_IO0, MountingHole:MountingHole_2.2mm_M2_DIN965_Pad_TopBottom, symbol Mechanical:MountingHole_Pad
- added H16: DA1_I2, MountingHole:MountingHole_2.2mm_M2_DIN965_Pad_TopBottom, symbol Mechanical:MountingHole_Pad
- added H17: GND, MountingHole:MountingHole_2.2mm_M2_DIN965_Pad_TopBottom, symbol Mechanical:MountingHole_Pad
- added H18: DA2C_IO2, MountingHole:MountingHole_2.2mm_M2_DIN965_Pad_TopBottom, symbol Mechanical:MountingHole_Pad
- added H19: DA2T_IO3, MountingHole:MountingHole_2.2mm_M2_DIN965_Pad_TopBottom, symbol Mechanical:MountingHole_Pad
- added H2: Ext3.3V_POWER, MountingHole:MountingHole_2.2mm_M2_DIN965_Pad_TopBottom, symbol Mechanical:MountingHole_Pad
- added H20: DA2T_IO1, MountingHole:MountingHole_2.2mm_M2_DIN965_Pad_TopBottom, symbol Mechanical:MountingHole_Pad
- added H21: DA1_I3, MountingHole:MountingHole_2.2mm_M2_DIN965_Pad_TopBottom, symbol Mechanical:MountingHole_Pad
- added H22: DA1_I1, MountingHole:MountingHole_2.2mm_M2_DIN965_Pad_TopBottom, symbol Mechanical:MountingHole_Pad
- added H3: D_IO1, MountingHole:MountingHole_2.2mm_M2_DIN965_Pad_TopBottom, symbol Mechanical:MountingHole_Pad
- added H4: D_IO2, MountingHole:MountingHole_2.2mm_M2_DIN965_Pad_TopBottom, symbol Mechanical:MountingHole_Pad
- added H5: D_IO3, MountingHole:MountingHole_2.2mm_M2_DIN965_Pad_TopBottom, symbol Mechanical:MountingHole_Pad
- added H6: D_IO4, MountingHole:MountingHole_2.2mm_M2_DIN965_Pad_TopBottom, symbol Mechanical:MountingHole_Pad
- added H7: D_IO5, MountingHole:MountingHole_2.2mm_M2_DIN965_Pad_TopBottom, symbol Mechanical:MountingHole_Pad
- added H8: D_IO6, MountingHole:MountingHole_2.2mm_M2_DIN965_Pad_TopBottom, symbol Mechanical:MountingHole_Pad
- added H9: DA1T_IO0, MountingHole:MountingHole_2.2mm_M2_DIN965_Pad_TopBottom, symbol Mechanical:MountingHole_Pad
- added Q1, Q2, Q3: PMOS, Package_TO_SOT_SMD:SuperSOT-3, symbol Simulation_SPICE:PMOS
- added R10, R3, R4: 100KΩ, Resistor_SMD:R_0201_0603Metric, symbol Device:R_US
- C1, C2, C3, C4, C5, C6, C9: footprint (none) -> Capacitor_Tantalum_SMD:CP_EIA-1608-10_AVX-L
- C7, C8: footprint Capacitor_THT:CP_Axial_L10.0mm_D4.5mm_P15.00mm_Horizontal -> Capacitor_Tantalum_SMD:CP_EIA-1608-10_AVX-L
- D1: footprint (none) -> LED_SMD:LED_0201_0603Metric
- D2: footprint Diode_SMD:D_SMA -> Diode_SMD:D_0603_1608Metric_Pad1.05x0.95mm_HandSolder
- F1: footprint (none) -> Fuse:Fuse_0603_1608Metric
- J2: footprint (none) -> Connector_PinHeader_2.54mm:PinHeader_1x06_P2.54mm_Vertical
- P1: footprint (none) -> Connector_USB:USB_C_Receptacle_GCT_USB4085
- R1, R2, R5, R6, R7, R8, R9: footprint Resistor_THT:R_Axial_DIN0207_L6.3mm_D2.5mm_P15.24mm_Horizontal -> Resistor_SMD:R_0201_0603Metric
Connections:
- net Vcc3.3V is gone; now on net Vcc3.3V_POWER: C2.1, D1.2 (A), U3.2 (VO)
- net DA1T_IO0: now also H9.1
- net DA1T_IO1: now also H10.1
- net DA1_I0: now also H11.1
- net DA1_I1: now also H22.1
- net DA1_I2: now also H16.1
- net DA1_I3: now also H21.1
- net DA2C_IO1: now also H13.1
- net DA2C_IO2: now also H18.1
- net DA2T_IO0: now also H15.1
- net DA2T_IO1: now also H20.1
- net DA2T_IO2: now also H14.1
- net DA2T_IO3: now also H19.1
- net D_IO0: now also H1.1
- net D_IO1: now also H3.1
- net D_IO2: now also H4.1
- net D_IO3: now also H5.1
- net D_IO4: now also H6.1
- net D_IO5: now also H7.1
- net D_IO6: now also H8.1
- net GND: now also H17.1
- net 3.3V renamed Vcc3.3V_POWER
- net Vcc3.3V_POWER: now also Q3.1 (D), Q3.2 (G), R3.1
- net LDOin renamed VREG_IN_POWER
- net VREG_IN_POWER: now also Q1.1 (D), Q1.2 (G), Q2.1 (D), Q2.2 (G), R10.1, R4.1
- net VBUS renamed USB_POWER
- net USB_POWER: now also Q2.3 (S), R4.2
- net Vin renamed Barrel_POWER
- net Barrel_POWER: now also Q1.3 (S), R10.2
- new net Ext3.3V_POWER: H2.1, Q3.3 (S), R3.2
Other:
- note added: "Power Switching"
- note removed: "Jumper Connections"
- moved on the sheet: C2, C3, C4, D1, J2, R5, U3
