File: School Projects/Conveyor_Belt_Arduino_mega_board/Conveyor_Belt_Arduino_mega_board.kicad_sch (KiCad schematic)
At the start: 24 parts, among them J1 Conn_01x08_Pin, J2 Conn_01x08_Pin, J3 Conn_01x08_Pin, J4 Conn_01x08_Pin, J5 Conn_01x08_Pin, J6 Conn_01x10_Pin, J7 SM04B-SRSS-TB

Commit message: Removed some unnecessary parts like reset button and emergency stop based on final production board
Parts:
- removed Creset1: 0.1uF, Capacitor_THT:CP_Axial_L10.0mm_D4.5mm_P15.00mm_Horizontal, symbol Device:C_US
- removed PUSH_BUTTON1: ~, TerminalBlock_Phoenix:TerminalBlock_Phoenix_MKDS-1,5-2_1x02_P5.00mm_Horizontal, symbol Connector:Screw_Terminal_01x02
- removed REST_BUTTON1: RST_BTN, Button_Switch_THT:SW_PUSH_6mm, symbol Switch:SW_Push
- removed Rresetmcu1, Rssbutton1: 10KΩ, Resistor_THT:R_Axial_DIN0309_L9.0mm_D3.2mm_P12.70mm_Horizontal, symbol Device:R_US
Connections:
- net IR_IN: now also J6.7 (Pin_7); no longer J6.9 (Pin_9)
- net Reset: no longer names the net of J1.3 (Pin_3)
- net S/S button: no longer names the net of J4.5 (Pin_5)
Other:
- note added: "MOTOR DRIVER CONNECTIONS"
- note removed: "RESET BUTTON"
- note removed: "START/STOP BUTTON"
- note removed: "TB66000 CONNECTIONS"
- moved on the sheet: BUCK_IN1, BUCK_OUT1, Cpw1, Cpw2, D1, Fuse1, J1, J2, J3, J4, J5, J6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
